File: circuit/focuser/focuser.kicad_sch (KiCad schematic)
At the start: 4 parts, among them M1 Stepper_Motor_bipolar, U1 Pico, U2 TMC2209_SILENTSTEPSTICK

Commit message: Updating circuit diagram with the optional manual switches
Parts:
- added SW1, SW2: SW_Push, symbol Switch:SW_Push
Connections:
- net at U1.25 (GPIO19): now also SW1.2
- net at U1.26 (GPIO20): now also SW2.2
- net at U1.42 (GND): now also SW1.1, SW2.1
Other:
- note added: "100uF 50v"
- note added: "Optional Manual Inputs, Increase / Decrease focus"
Changed lines of the file:
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@@
   (title_block
     (title "D.I.Y. Moonlyte focuser")
-    (date "2023-10-19")
-    (rev "1")
+    (date "2023-11-03")
+    (rev "2")
     (company "John Knight")
   )
@@
   (junction (at 165.1 146.05) (diameter 0) (color 0 0 0 0)
   )
+  (junction (at 92.71 165.1) (diameter 0) (color 0 0 0 0)
+  )
   (junction (at 187.96 146.05) (diameter 0) (color 0 0 0 0)
   )
@@
     (stroke (width 0) (type default))
   )
+  (wire (pts (xy 92.71 144.78) (xy 92.71 165.1))
+    (stroke (width 0) (type default))
+  )
   (wire (pts (xy 148.59 111.76) (xy 170.18 111.76))
     (stroke (width 0) (type default))
@@
     (stroke (width 0) (type default))
   )
+  (wire (pts (xy 92.71 165.1) (xy 92.71 179.07))
+    (stroke (width 0) (type default))
+  )
+  (wire (pts (xy 92.71 165.1) (xy 97.79 165.1))
+    (stroke (width 0) (type default))
+  )
   (wire (pts (xy 142.24 101.6) (xy 110.49 101.6))
     (stroke (width 0) (type default))
@@
     (stroke (width 0) (type default))
   )
+  (wire (pts (xy 110.49 129.54) (xy 121.92 129.54))
+    (stroke (width 0) (type default))
+  )
   (wire (pts (xy 110.49 137.16) (xy 148.59 137.16))
     (stroke (width 0) (type default))
@@
     (stroke (width 0) (type default))
   )
+  (wire (pts (xy 92.71 179.07) (xy 97.79 179.07))
+    (stroke (width 0) (type default))
+  )
   (wire (pts (xy 148.59 137.16) (xy 148.59 111.76))
     (stroke (width 0) (type default))
@@
     (stroke (width 0) (type default))
   )
+  (wire (pts (xy 110.49 127) (xy 127 127))
+    (stroke (width 0) (type default))
+  )
   (wire (pts (xy 146.05 104.14) (xy 170.18 104.14))
     (stroke (width 0) (type default))
   )
+  (wire (pts (xy 107.95 179.07) (xy 127 179.07))
+    (stroke (width 0) (type default))
+  )
   (wire (pts (xy 205.74 119.38) (xy 242.57 119.38))
     (stroke (width 0) (type default))
   )
+  (wire (pts (xy 121.92 129.54) (xy 121.92 165.1))
+    (stroke (width 0) (type default))
+  )
   (wire (pts (xy 170.18 119.38) (xy 165.1 119.38))
     (stroke (width 0) (type default))
@@
     (stroke (width 0) (type default))
   )
+  (wire (pts (xy 107.95 165.1) (xy 121.92 165.1))
+    (stroke (width 0) (type default))
+  )
   (wire (pts (xy 250.19 109.22) (xy 232.41 109.22))
     (stroke (width 0) (type default))
@@
     (stroke (width 0) (type default))
   )
+  (wire (pts (xy 127 127) (xy 127 179.07))
+    (stroke (width 0) (type default))
+  )
   (wire (pts (xy 110.49 132.08) (xy 146.05 132.08))
     (stroke (width 0) (type default))
@@
   (wire (pts (xy 227.33 93.98) (xy 215.9 93.98))
     (stroke (width 0) (type default))
+  )
+  (text "100uF 50v" (at 243.84 97.79 0)
+    (effects (font (size 1.27 1.27)) (justify left bottom))
+  )
+  (text "Optional Manual Inputs,\nIncrease / Decrease focus" (at 64.77 171.45 0)
+    (effects (font (size 1.27 1.27)) (justify left bottom))
   )
   (symbol (lib_id "power:+12V") (at 262.89 93.98 0) (unit 1)
@@
         (path "/e4734da5-82cd-4c77-b1d9-aed07072de3f"
           (reference "C1") (unit 1)
+        )
+      )
+    )
+  )
+  (symbol (lib_id "Switch:SW_Push") (at 102.87 165.1 0) (unit 1)
+    (in_bom yes) (on_board yes) (dnp no) (fields_autoplaced)
+    (property "Reference" "SW1" (at 102.87 157.48 0)
+      (effects (font (size 1.27 1.27)))
+    )
+    (property "Value" "SW_Push" (at 102.87 160.02 0)
+      (effects (font (size 1.27 1.27)))
+    )
+    (property "Footprint" "" (at 102.87 160.02 0)
+      (effects (font (size 1.27 1.27)) hide)
+    )
+    (property "Datasheet" "~" (at 102.87 160.02 0)
+      (effects (font (size 1.27 1.27)) hide)
+    )
+    (pin "1")
+    (pin "2")
+    (instances
+      (project "focuser"
+        (path "/e4734da5-82cd-4c77-b1d9-aed07072de3f"
+          (reference "SW1") (unit 1)
         )
       )
@@
         )
       )
+    )
+  )
+  (symbol (lib_id "Switch:SW_Push") (at 102.87 179.07 0) (unit 1)
+    (in_bom yes) (on_board yes) (dnp no) (fields_autoplaced)
+    (property "Reference" "SW2" (at 102.87 171.45 0)
+      (effects (font (size 1.27 1.27)))
+    )
+    (property "Value" "SW_Push" (at 102.87 173.99 0)
+      (effects (font (size 1.27 1.27)))
+    )
+    (property "Footprint" "" (at 102.87 173.99 0)
+      (effects (font (size 1.27 1.27)) hide)
+    )
+    (property "Datasheet" "~" (at 102.87 173.99 0)
+      (effects (font (size 1.27 1.27)) hide)
+    )
+    (pin "1")
+    (pin "2")
+    (instances
+      (project "focuser"
+        (path "/e4734da5-82cd-4c77-b1d9-aed07072de3f"
+          (reference "SW2") (unit 1)
+        )
+      )
